File: KiCad/ArmchairBarf.kicad_pcb (KiCad board)
At the start: 2 copper layers, 13.3 x 11.6 mm, 10 parts, among them J1 Conn_01x03_Socket, J2 Conn_01x03_Socket, U1 WS2812-2020, U2 WS2812-2020, U3 WS2812-2020, U4 WS2812-2020, U5 WS2812-2020, U6 WS2812-2020

Commit message: V1 release!
Routing:
- net Net-(U4-DO): track 2.80 -> 3.59 mm
Changed lines of the file:
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@@
     (property "Sheetname" "")
     (attr smd)
-    (fp_text reference "U1" (at 0.517 -1.86247) (layer "F.SilkS")
+    (fp_text reference "U1" (at 0.517 -1.86247) (layer "F.SilkS") hide
         (effects (font (size 0.64 0.64) (thickness 0.15)))
     )
@@
     (property "ki_keywords" "cap capacitor")
     (attr smd)
-    (fp_text reference "C1" (at 0 -1.16) (layer "F.SilkS")
+    (fp_text reference "C1" (at 0 -1.16) (layer "F.SilkS") hide
         (effects (font (size 1 1) (thickness 0.15)))
     )
@@
     (property "ki_keywords" "R res resistor")
     (attr smd)
-    (fp_text reference "R1" (at 0 -1.17) (layer "F.SilkS")
+    (fp_text reference "R1" (at 0 -1.17) (layer "F.SilkS") hide
         (effects (font (size 1 1) (thickness 0.15)))
     )
@@
     (property "Sheetname" "")
     (attr smd)
-    (fp_text reference "U6" (at 0.517 -1.86247) (layer "F.SilkS")
+    (fp_text reference "U6" (at 0.517 -1.86247) (layer "F.SilkS") hide
         (effects (font (size 0.64 0.64) (thickness 0.15)))
     )
@@
     (property "Sheetname" "")
     (attr smd)
-    (fp_text reference "U4" (at 0.517 -1.86247) (layer "F.SilkS")
+    (fp_text reference "U4" (at 0.517 -1.86247) (layer "F.SilkS") hide
         (effects (font (size 0.64 0.64) (thickness 0.15)))
     )
@@
     (property "Sheetname" "")
     (attr smd)
-    (fp_text reference "U3" (at 2.351389 -0.626504) (layer "F.SilkS")
+    (fp_text reference "U3" (at 2.351389 -0.626504) (layer "F.SilkS") hide
         (effects (font (size 0.64 0.64) (thickness 0.15)))
     )
@@
     (property "Sheetname" "")
     (attr smd)
-    (fp_text reference "U2" (at 0.517 -1.86247) (layer "F.SilkS")
+    (fp_text reference "U2" (at 0.517 -1.86247) (layer "F.SilkS") hide
         (effects (font (size 0.64 0.64) (thickness 0.15)))
     )
@@
     (property "Sheetname" "")
     (attr smd)
-    (fp_text reference "U5" (at 0.517 -1.86247) (layer "F.SilkS")
+    (fp_text reference "U5" (at 0.517 -1.86247) (layer "F.SilkS") hide
         (effects (font (size 0.64 0.64) (thickness 0.15)))
     )
@@
   (segment (start 151.69 98.89) (end 152.395 98.89) (width 0.25) (layer "F.Cu") (net 5))
   (segment (start 155.5 105.875) (end 155.75 105.875) (width 0.25) (layer "F.Cu") (net 6))
-  (segment (start 158.08 103.639994) (end 158.08 100.29) (width 0.25) (layer "F.Cu") (net 6))
+  (segment (start 158.08 102.675586) (end 158.08 100.29) (width 0.25) (layer "F.Cu") (net 6))
+  (segment (start 157.460891 104.36724) (end 157.885586 103.942545) (width 0.25) (layer "F.Cu") (net 6))
+  (segment (start 158.08 100.29) (end 156.68 98.89) (width 0.25) (layer "F.Cu") (net 6))
+  (segment (start 157.885586 103.942545) (end 157.885586 102.87) (width 0.25) (layer "F.Cu") (net 6))
+  (segment (start 155.75 105.875) (end 157.25776 104.36724) (width 0.25) (layer "F.Cu") (net 6))
+  (segment (start 157.25776 104.36724) (end 157.460891 104.36724) (width 0.25) (layer "F.Cu") (net 6))
+  (segment (start 157.885586 102.87) (end 158.08 102.675586) (width 0.25) (layer "F.Cu") (net 6))
   (segment (start 156.68 98.89) (end 155.575 98.89) (width 0.25) (layer "F.Cu") (net 6))
-  (segment (start 158.08 100.29) (end 156.68 98.89) (width 0.25) (layer "F.Cu") (net 6))
-  (segment (start 156.85 104.775) (end 157.433952 104.775) (width 0.25) (layer "F.Cu") (net 6))
-  (segment (start 157.433952 104.775) (end 158.08 103.639994) (width 0.25) (layer "F.Cu") (net 6))
-  (segment (start 155.75 105.875) (end 156.85 104.775) (width 0.25) (layer "F.Cu") (net 6))
+  (segment (start 157.405 102.065) (end 157.015 102.065) (width 0.25) (layer "F.Cu") (net 7))
+  (segment (start 156.845 102.235) (end 156.845 102.91) (width 0.25) (layer "F.Cu") (net 7))
+  (segment (start 154.825 104.775) (end 153.67 104.775) (width 0.25) (layer "F.Cu") (net 7))
+  (segment (start 157.015 102.065) (end 156.845 102.235) (width 0.25) (layer "F.Cu") (net 7))
   (segment (start 155.655 104.1) (end 154.825 104.1) (width 0.25) (layer "F.Cu") (net 7))
-  (segment (start 156.25 103.505) (end 155.655 104.1) (width 0.25) (layer "F.Cu") (net 7))
+  (segment (start 156.845 102.91) (end 155.655 104.1) (width 0.25) (layer "F.Cu") (net 7))
   (segment (start 154.825 104.1) (end 154.825 104.775) (width 0.25) (layer "F.Cu") (net 7))
-  (segment (start 156.25 102.195) (end 156.25 103.505) (width 0.25) (layer "F.Cu") (net 7))
-  (segment (start 157.405 102.065) (end 156.38 102.065) (width 0.25) (layer "F.Cu") (net 7))
-  (segment (start 154.825 104.775) (end 153.67 104.775) (width 0.25) (layer "F.Cu") (net 7))
-  (segment (start 156.38 102.065) (end 156.25 102.195) (width 0.25) (layer "F.Cu") (net 7))
-  (segment (start 154.27 101.0175) (end 154.27 101.64) (width 0.25) (layer "F.Cu") (net 8))
-  (segment (start 155.575 100.965) (end 154.3225 100.965) (width 0.25) (layer "F.Cu") (net 8))
-  (segment (start 153.845 102.065) (end 153.595 102.065) (width 0.25) (layer "F.Cu") (net 8))
-  (segment (start 154.3225 100.965) (end 154.27 101.0175) (width 0.25) (layer "F.Cu") (net 8))
-  (segment (start 154.27 101.64) (end 153.845 102.065) (width 0.25) (layer "F.Cu") (net 8))
+  (segment (start 155.334224 100.724224) (end 154.333592 100.724224) (width 0.25) (layer "F.Cu") (net 8))
+  (segment (start 154.305 100.752816) (end 154.305 101.605) (width 0.25) (layer "F.Cu") (net 8))
+  (segment (start 155.575 100.965) (end 155.334224 100.724224) (width 0.25) (layer "F.Cu") (net 8))
+  (segment (start 153.67 101.64) (end 153.595 101.715) (width 0.25) (layer "F.Cu") (net 8))
+  (segment (start 154.333592 100.724224) (end 154.305 100.752816) (width 0.25) (layer "F.Cu") (net 8))
+  (segment (start 155.575 100.965) (end 155.325 100.965) (width 0.25) (layer "F.Cu") (net 8))
+  (segment (start 154.305 101.605) (end 154.27 101.64) (width 0.25) (layer "F.Cu") (net 8))
+  (segment (start 154.27 101.64) (end 153.67 101.64) (width 0.25) (layer "F.Cu") (net 8))
+  (segment (start 153.595 101.715) (end 153.595 102.065) (width 0.25) (layer "F.Cu") (net 8))
   (segment (start 151.765 100.965) (end 151.165 100.965) (width 0.25) (layer "F.Cu") (net 9))
   (segment (start 150.065 102.065) (end 149.785 102.065) (width 0.25) (layer "F.Cu") (net 9))

Commit message: Cleanup of V1
Other:
- board text added: "By Lilliana"
Changed lines of the file:
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@@
       (drillshape 0)
       (scaleselection 1)
-      (outputdirectory "")
+      (outputdirectory "../Gerber/")
     )
   )
@@
     )
     (stroke (width 0.1) (type solid)) (fill none) (layer "Edge.Cuts"))
+  (gr_text "By Lilliana\n" (at 156.253793 105.048706 270) (layer "B.SilkS")
+    (effects (font (size 0.8 0.8) (thickness 0.1) bold) (justify left bottom mirror))
+  )
   (segment (start 149.055 99.695) (end 149.86 98.89) (width 0.25) (layer "F.Cu") (net 1))
   (segment (start 154.633897 99.778897) (end 153.745 98.89) (width 0.25) (layer "F.Cu") (net 1))
